File: rev_b/bus_grove12.kicad_pcb (KiCad board)
At the start: 2 copper layers, 100 x 100 mm, 113 parts, among them J1 TERMINATE_JUMPER, J2 LED_CONN_2X2, SW1 MJTP1243, U1 LM2940, U2 74HCT08, U3 MCP2562, U4 74HCT03, U5 ATMEGA328_DIP28, X1 16MHz

Commit message: Rev. B is ready.
Connections:
- net VCC renamed +5V
- H1 pad 1: GND -> (no net)
- H10 pad 1: GND -> (no net)
- H11 pad 1: GND -> (no net)
- H12 pad 1: GND -> (no net)
- H13 pad 1: GND -> (no net)
- H14 pad 1: GND -> (no net)
- H15 pad 1: GND -> (no net)
- H16 pad 1: GND -> (no net)
- H17 pad 1: GND -> (no net)
- H18 pad 1: GND -> (no net)
- H19 pad 1: GND -> (no net)
- H2 pad 1: GND -> (no net)
- H20 pad 1: GND -> (no net)
- H21 pad 1: GND -> (no net)
- H22 pad 1: GND -> (no net)
- H23 pad 1: GND -> (no net)
- H24 pad 1: GND -> (no net)
- H25 pad 1: GND -> (no net)
- H26 pad 1: GND -> (no net)
- H27 pad 1: GND -> (no net)
- H28 pad 1: GND -> (no net)
- H29 pad 1: GND -> (no net)
- H3 pad 1: GND -> (no net)
- H30 pad 1: GND -> (no net)
- H31 pad 1: GND -> (no net)
- H32 pad 1: GND -> (no net)
- H33 pad 1: GND -> (no net)
- H34 pad 1: GND -> (no net)
- H35 pad 1: GND -> (no net)
- H36 pad 1: GND -> (no net)
- H37 pad 1: GND -> (no net)
- H38 pad 1: GND -> (no net)
- H39 pad 1: GND -> (no net)
- H4 pad 1: GND -> (no net)
- H40 pad 1: GND -> (no net)
- H41 pad 1: GND -> (no net)
- H42 pad 1: GND -> (no net)
- H43 pad 1: GND -> (no net)
- H44 pad 1: GND -> (no net)
- H45 pad 1: GND -> (no net)
- H46 pad 1: GND -> (no net)
- H47 pad 1: GND -> (no net)
- H48 pad 1: GND -> (no net)
- H49 pad 1: GND -> (no net)
- H5 pad 1: GND -> (no net)
- H50 pad 1: GND -> (no net)
- H51 pad 1: GND -> (no net)
- H52 pad 1: GND -> (no net)
- H53 pad 1: GND -> (no net)
- H54 pad 1: GND -> (no net)
- H55 pad 1: GND -> (no net)
- H56 pad 1: GND -> (no net)
- H57 pad 1: GND -> (no net)
- H58 pad 1: GND -> (no net)
- H59 pad 1: GND -> (no net)
- H6 pad 1: GND -> (no net)
- H60 pad 1: GND -> (no net)
- H7 pad 1: GND -> (no net)
- H8 pad 1: GND -> (no net)
- H9 pad 1: GND -> (no net)
- R9 pad 2: Net-(R9-Pad2) -> Net-(C7-Pad1)
- U4 pad 12: Net-(R9-Pad2) -> Net-(C7-Pad1)
- U4 pad 13: Net-(R9-Pad2) -> Net-(C7-Pad1)
Routing:
- net Net-(C7-Pad1): track 3.44 -> 38.0 mm
- net Net-(R9-Pad2): track 15.0 -> 0.00 mm
Other:
- board text added: "BUS_GROVE12 REV. B 9FEB2015 (C) 2014 GRAMLICH"
- board text removed: "bus_grove12 Rev. A 2Nov2014 (c) 2014 by Gramlich"
