File: rev_b/holes.sch (KiCad schematic (older format))
At the start: 56 parts

Commit message: Rev. B is ready.
Connections:
- removed net GND: H10.1 (GND), H11.1 (GND), H12.1 (GND), H13.1 (GND), H14.1 (GND), H15.1 (GND), H16.1 (GND), H17.1 (GND), H18.1 (GND), H19.1 (GND), H20.1 (GND), H21.1 (GND)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
- no-connect marks 0 -> 56
